File: engine_start_battery.sch (KiCad schematic (older format))
At the start: 4 parts

Commit message: Several updates, maybe final version for season 2021
Parts:
- removed Engine_Alternator: Engine alternator, symbol Connector_Generic:Conn_01x03
- removed Engine_charge_distributor: Sterling model X, symbol Connector_Generic:Conn_2Rows-05Pins
- added Alternator_charge_distribition: Alternator charging distribution / Sterling ProSp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, symbol Simple_connector:No_pin_nums_5_conns
- added Engine_Alternator: Engine alternator, symbol Connector_Generic:Conn_01x02
Connections:
- net GND: now also Alternator_charge_distribition.5 (Pin_5), Engine_Alternator.2 (Pin_2)
- net Engine_Power_Input renamed Engine
- net Engine_charge_distribution_2 renamed Charge_distribution_start
- net Charge_distribution_start: now also Alternator_charge_distribition.4 (Pin_4)
- new net Alt_In: Alternator_charge_distribition.1 (Pin_1), Engine_Alternator.1 (Pin_1)
- new net Charge_distribution_house: Alternator_charge_distribition.2 (Pin_2)
- new net Pos_Ign_feed: Alternator_charge_distribition.3 (Pin_3)
Changed lines of the file:
@@
 Sheet 4 5
 Title "S/Y Kaisla - engine start battery & charge distribution"
-Date "2021-03-14"
+Date "2021-04-04"
 Rev "1"
 Comp "Jukka Aittola"
@@
 	5400 1500 6900 1500
 Text GLabel 6900 1500 2    50   Input ~ 0
-Engine_Power_Input
+Engine
 Wire Wire Line
 	2000 1500 2900 1500
@@
 	4100 1500 5000 1500
 Text GLabel 4100 2050 3    50   Input ~ 0
-Engine_charge_distribution_2
+Charge_distribution_start
 Text GLabel 3500 2050 3    50   Input ~ 0
 Shore_power_charge_2
@@
 Wire Wire Line
 	2000 3500 2000 2650
-$Comp
-L Connector_Generic:Conn_01x03 Engine_Alternator
-U 1 1 604EC83E
-P 2000 4650
-F 0 "Engine_Alternator" H 1918 4875 50  0000 C CNN
-F 1 "Engine alternator" H 1918 4876 50  0001 C CNN
-F 2 "" H 2000 4650 50  0001 C CNN
-F 3 "~" H 2000 4650 50  0001 C CNN
-	1    2000 4650
-	-1   0    0    -1
-$EndComp
-$Comp
-L Connector_Generic:Conn_2Rows-05Pins Engine_charge_distributor
-U 1 1 604EE6E0
-P 4950 4650
-F 0 "Engine_charge_distributor" H 5000 4967 50  0000 C CNN
-F 1 "Sterling model X" H 5000 4876 50  0000 C CNN
-F 2 "" H 4950 4650 50  0001 C CNN
-F 3 "~" H 4950 4650 50  0001 C CNN
-	1    4950 4650
-	1    0    0    -1
-$EndComp
 Wire Wire Line
 	2200 4550 4750 4550
-Wire Wire Line
-	4750 4650 2200 4650
 $Comp
 L power:GND #PWR?
@@
 	4750 5150 4750 4750
 Wire Wire Line
-	2200 5150 2200 4750
+	2200 5150 2200 4650
 Text Label 2400 4550 0    50   ~ 0
 Alternator+
-Text Label 2400 4650 0    50   ~ 0
-Alternator_sense
 Wire Wire Line
 	5250 4550 6050 4550
@@
 	5250 4650 6050 4650
 Text GLabel 6050 4550 2    50   Input ~ 0
-Engine_charge_distribution_1
+Charge_distribution_house
 Text GLabel 6050 4650 2    50   Input ~ 0
-Engine_charge_distribution_2
+Charge_distribution_start
 Connection ~ 2900 1500
 Wire Wire Line
@@
 	2900 1500 2900 2050
 Text GLabel 2900 2050 3    50   Input ~ 0
-U_meas_1
+U_meas_start
+$Comp
+L Simple_connector:No_pin_nums_5_conns Alternator_charge_distribition
+U 1 1 606E0CFC
+P 4950 4650
+F 0 "Alternator_charge_distribition" H 5000 4967 50  0001 C CNN
+F 1 "Alternator charging distribution / Sterling ProSplit R" H 5000 4875 50  0000 C CNN
+F 2 "" H 4950 4650 50  0001 C CNN
+F 3 "~" H 4950 4650 50  0001 C CNN
+	1    4950 4650
+	1    0    0    -1
+$EndComp
+$Comp
+L Connector_Generic:Conn_01x02 Engine_Alternator
+U 1 1 606E2FAC
+P 2000 4550
+F 0 "Engine_Alternator" H 1918 4767 50  0001 C CNN
+F 1 "Engine alternator" H 1918 4675 50  0000 C CNN
+F 2 "" H 2000 4550 50  0001 C CNN
+F 3 "~" H 2000 4550 50  0001 C CNN
+	1    2000 4550
+	-1   0    0    -1
+$EndComp
+Text Label 4350 4550 2    50   ~ 0
+Alt_In
+Text GLabel 4350 4650 0    50   Input ~ 0
+Pos_Ign_feed
+Wire Wire Line
+	4750 4650 4350 4650
+Text Label 5400 4550 0    50   ~ 0
+Batt_2
+Text Label 5425 4650 0    50   ~ 0
+Start_Batt
 $EndSCHEMATC
