File: house_batteries.sch (KiCad schematic (older format))
At the start: 10 parts

Commit message: Several updates, maybe final version for season 2021
Parts:
- removed Power_Monitor: Sterling Power Monitor, symbol Connector_Generic:Conn_01x07
- added Sterling_power_monitor: Sterling Power Management Panel, symbol Simple_connector:No_pin_nums_6_conns
- F1: renamed from F_1_1; value 20A (?) -> 15A
- F_1_2: value 5A (?) -> 20A
- F_1_4: value 5A (?) -> 10A
Connections:
- net GND: now also Sterling_power_monitor.1 (Pin_1)
- net R_shunt_1: now also Sterling_power_monitor.2 (Pin_2), Sterling_power_monitor.4 (Pin_4), Sterling_power_monitor.5 (Pin_5)
- net Engine_charge_distribution_1 renamed Charge_distribution_house
- net Charge_distribution_house: now also Sterling_power_monitor.6 (Pin_6)
- new net U_meas_start: Sterling_power_monitor.3 (Pin_3)
Changed lines of the file:
@@
 Sheet 3 5
 Title "S/Y Kaisla - house battery bank"
-Date "2021-03-14"
+Date "2021-04-04"
 Rev "1"
 Comp "Jukka Aittola"
@@
 Text GLabel 3950 2500 3    50   Input ~ 0
 Shore_power_charge_1
-Text GLabel 4700 2500 3    50   Input ~ 0
-Engine_charge_distribution_1
-$Comp
-L Device:Fuse F_1_1
+$Comp
+L Device:Fuse F1
 U 1 1 604F8550
 P 5700 2650
-F 0 "F_1_1" H 5760 2696 50  0000 L CNN
-F 1 "20A (?)" H 5760 2605 50  0000 L CNN
+F 0 "F1" H 5760 2696 50  0001 L CNN
+F 1 "15A" H 5760 2605 50  0000 L CNN
 F 2 "" V 5630 2650 50  0001 C CNN
 F 3 "~" H 5700 2650 50  0001 C CNN
@@
 U 1 1 604FA099
 P 6150 2650
-F 0 "F_1_2" H 6210 2696 50  0000 L CNN
-F 1 "5A (?)" H 6210 2605 50  0000 L CNN
+F 0 "F_1_2" H 6210 2696 50  0001 L CNN
+F 1 "20A" H 6210 2605 50  0000 L CNN
 F 2 "" V 6080 2650 50  0001 C CNN
 F 3 "~" H 6150 2650 50  0001 C CNN
@@
 L Device:Fuse F_1_4
 U 1 1 604FA4CD
-P 6850 2650
-F 0 "F_1_4" H 6910 2696 50  0000 L CNN
-F 1 "5A (?)" H 6910 2605 50  0000 L CNN
-F 2 "" V 6780 2650 50  0001 C CNN
-F 3 "~" H 6850 2650 50  0001 C CNN
-	1    6850 2650
+P 6625 2650
+F 0 "F_1_4" H 6685 2696 50  0001 L CNN
+F 1 "10A" H 6685 2605 50  0000 L CNN
+F 2 "" V 6555 2650 50  0001 C CNN
+F 3 "~" H 6625 2650 50  0001 C CNN
+	1    6625 2650
 	1    0    0    -1
 $EndComp
@@
 	5700 2500 6150 2500
 Wire Wire Line
-	6150 2500 6850 2500
+	6150 2500 6625 2500
 Connection ~ 6150 2500
 Wire Wire Line
@@
 	1    0    0    -1
 $EndComp
-Wire Wire Line
-	6850 2800 6850 3600
 $Comp
 L power:GND #PWR?
@@
 Wire Notes Line
 	5300 2100 5300 3300
-Wire Notes Line
-	5300 3300 7300 3300
-Wire Notes Line
-	7300 3300 7300 2100
-Wire Notes Line
-	7300 2100 5300 2100
 $Comp
 L Switch:SW_SPST Main_Switch_1
@@
 	1    0    0    -1
 $EndComp
-Wire Wire Line
-	2000 1750 2500 1750
 Connection ~ 2000 1750
-$Comp
-L Connector_Generic:Conn_01x07 Power_Monitor
-U 1 1 60523C0C
-P 1500 5350
-F 0 "Power_Monitor" H 1418 5867 50  0000 C CNN
-F 1 "Sterling Power Monitor" H 1418 5776 50  0000 C CNN
-F 2 "" H 1500 5350 50  0001 C CNN
-F 3 "~" H 1500 5350 50  0001 C CNN
-	1    1500 5350
+Text GLabel 2500 1750 3    50   Input ~ 0
+U_meas_house
+Text GLabel 2175 5400 2    50   Input ~ 0
+U_meas_house
+Text GLabel 2175 5300 2    50   Input ~ 0
+U_meas_start
+Text GLabel 2175 5600 2    50   Input ~ 0
+R_shunt_2
+Text GLabel 2175 5500 2    50   Input ~ 0
+R_shunt_1
+Wire Wire Line
+	2000 1750 3050 1750
+Wire Wire Line
+	6625 2800 6625 3600
+Wire Wire Line
+	6625 3600 6850 3600
+Wire Notes Line
+	5300 2100 6900 2100
+Wire Notes Line
+	6900 2100 6900 3300
+Wire Notes Line
+	6900 3300 5300 3300
+Text GLabel 4700 2500 3    50   Input ~ 0
+Charge_distribution_house
+$Comp
+L Simple_connector:No_pin_nums_6_conns Sterling_power_monitor
+U 1 1 606E634C
+P 1500 5300
+F 0 "Sterling_power_monitor" H 1418 5717 50  0001 C CNN
+F 1 "Sterling Power Management Panel" H 1418 5625 50  0000 C CNN
+F 2 "" H 1500 5300 50  0001 C CNN
+F 3 "~" H 1500 5300 50  0001 C CNN
+	1    1500 5300
 	-1   0    0    -1
 $EndComp
-Connection ~ 2500 1750
-Wire Wire Line
-	2500 1750 3050 1750
-Text GLabel 2500 1750 3    50   Input ~ 0
-U_meas_4
-Text GLabel 1700 5650 2    50   Input ~ 0
-U_meas_4
-Text GLabel 1700 5350 2    50   Input ~ 0
-U_meas_1
-Text GLabel 1700 5250 2    50   Input ~ 0
-R_shunt_2
-Text GLabel 1700 5150 2    50   Input ~ 0
-R_shunt_1
+Wire Wire Line
+	1700 5500 2175 5500
+Wire Wire Line
+	1700 5400 2175 5400
+Wire Wire Line
+	1700 5600 2175 5600
+Wire Wire Line
+	3350 5100 3350 5775
+Wire Wire Line
+	1700 5100 3350 5100
+$Comp
+L power:GND #PWR?
+U 1 1 606EEA76
+P 3350 5775
+F 0 "#PWR?" H 3350 5525 50  0001 C CNN
+F 1 "GND" H 3355 5602 50  0000 C CNN
+F 2 "" H 3350 5775 50  0001 C CNN
+F 3 "" H 3350 5775 50  0001 C CNN
+	1    3350 5775
+	1    0    0    -1
+$EndComp
+Text Label 1625 5100 0    50   ~ 0
+Power-
+Text Label 1625 5200 0    50   ~ 0
+Power+
+Text Label 1625 5300 0    50   ~ 0
+1A
+Text Label 1625 5400 0    50   ~ 0
+4A
+Text Label 1625 5500 0    50   ~ 0
+4B
+Text Label 1625 5600 0    50   ~ 0
+4C
+Wire Wire Line
+	1700 5300 2175 5300
+Text GLabel 2175 5200 2    50   Input ~ 0
+U_meas_house
+Wire Wire Line
+	1700 5200 2175 5200
 $EndSCHEMATC
