File: shore-power.sch (KiCad schematic (older format))
At the start: 10 parts

Commit message: Several updates, maybe final version for season 2021
Parts:
- removed CB_SP_2, CB_SP_3, CB_SP_4: Shore power circuit breaker, symbol Device:CircuitBreaker_2P
- removed SPC1: Shore power connector, symbol Connector_Generic:Conn_01x03
- removed SP_Out_1, SP_Out_2, SP_Out_3, SP_Out_4: Conn_01x03, symbol Connector_Generic:Conn_01x03
- added CB_SP_? (x3): Circuit breaker, symbol Device:CircuitBreaker_2P
- added J? (x5): Conn_Wallsocket_3pin_mod, symbol Simple_connector:Conn_Wallsocket_3pin_mod
- CB_SP_1: value Shore power circuit breaker -> Circuit breaker
Connections:
- net at RCD1.2: now also J?.1 (L)
- net at RCD1.4: now also J?.2 (N)
- net at CB_SP_1.1: now also J?.1 (L)
- net at CB_SP_1.3: now also J?.2 (N)
- net sp_L renamed L
- net L: now also CB_SP_?.2, CB_SP_?.2, CB_SP_?.2
- net sp_N renamed N
- net N: now also CB_SP_?.4, CB_SP_?.4, CB_SP_?.4
- new net: CB_SP_?.1, J?.1 (L) (x3)
- new net: CB_SP_?.3, J?.2 (N) (x3)
- new net PE: J?.3 (PE), J?.3 (PE), J?.3 (PE), J?.3 (PE), J?.3 (PE)
